File: tests.kicad_pcb (KiCad board)
At the start: 2 copper layers, 30 x 20 mm, 7 parts, among them J101 USB_A+C+XT30

Commit message: Moved footprint origin & added info  to README.md
Parts:
- moved J101 12.5 mm to (115.0, 100.0)
